File: kicad/SR-U2764.kicad_pcb (KiCad board)
At the start: 2 copper layers, 361.9 x 140.5 mm, 158 parts, among them SW1 SW_Push, SW10 SW_Push, SW11 SW_Push, SW12 SW_Push, SW13 SW_Push, SW14 SW_Push, SW15 SW_Push, SW16 SW_Push, SW17 SW_Push, SW18 SW_Push, SW19 SW_Push, SW2 SW_Push, SW20 SW_Push, SW21 SW_Push, SW22 SW_Push, SW23 SW_Push, SW24 SW_Push, SW25 SW_Push, SW26 SW_Push, SW27 SW_Push, SW28 SW_Push, SW29 SW_Push, SW3 SW_Push, SW30 SW_Push, SW31 SW_Push, SW32 SW_Push, SW33 SW_Push, SW34 SW_Push, SW35 SW_Push, SW36 SW_Push, SW37 SW_Push, SW38 SW_Push, SW39 SW_Push, SW4 SW_Push, SW40 SW_Push, SW41 SW_Push, SW42 SW_Push, SW43 SW_Push, SW44 SW_Push, SW45 SW_Push, SW46 SW_Push, SW47 SW_Push, SW48 SW_Push, SW49 SW_Push, SW5 SW_Push, SW50 SW_Push, SW51 SW_Push, SW52 SW_Push, SW53 SW_Push, SW54 SW_Push, SW55 SW_Push, SW56 SW_Push, SW57 SW_Push, SW58 SW_Push, SW59 SW_Push, SW6 SW_Push, SW60 SW_Push, SW61 SW_Push, SW62 SW_Push, SW63 SW_Push, SW64 SW_Push, SW65 SW_Push, SW66 SW_Push, SW67 SW_Push, SW68 SW_Push, SW69 SW_Push, SW7 SW_Push, SW70 SW_Push, SW71 SW_Push, SW72 SW_Push, SW73 SW_Push, SW74 SW_Push, SW75 SW_Push, SW76 SW_Push, SW77 SW_Push, SW78 SW_Push, SW8 SW_Push, SW9 SW_Push, U2 Pico

Commit message: update pcb and update journal
Routing:
- net COL8: track 417.7 -> 712.2 mm, vias 2 -> 4
- net COL5: track 559.7 -> 836.7 mm, vias 6 -> 9
- net COL6: track 337.9 -> 607.9 mm, vias 10 -> 14
- net ROW7: track 487.2 -> 719.0 mm
- net COL7: track 358.0 -> 572.0 mm, vias 4 -> 7
- net COL4: track 622.7 -> 806.7 mm, vias 9 -> 11
- net COL10: track 387.8 -> 566.6 mm, vias 8 -> 9
- net ROW1: track 210.9 -> 368.3 mm, vias 0 -> 8
- net COL9: track 475.9 -> 626.3 mm, vias 7 -> 11
- net ROW8: track 207.0 -> 346.8 mm
- net ROW4: track 171.4 -> 304.3 mm, vias 0 -> 4
- net ROW3: track 289.2 -> 408.8 mm, vias 0 -> 2
- net COL1: track 430.9 -> 549.6 mm, vias 5 -> 8
- net ROW6: track 252.5 -> 367.8 mm, vias 0 -> 4
- net ROW5: track 264.8 -> 372.6 mm, vias 0 -> 2
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